File: schlum-pcb/schlum-pcb/schlum-pcb.kicad_pcb (KiCad board)
At the start: 2 copper layers, 160 x 90 mm, 47 parts, among them IC1 TM1637__SOP_1, IC2 TM1637__SOP_1, J1 Screw_Terminal_01x03, J2 Conn_01x03_Male, J3 UART0_CONN, J4 Screw_Terminal_01x02, K1 SANYOU_SRD_Form_C, P1 RFID-RC522-MODULE, Q1 2N3904, U1 Optocoupler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

Commit message: Add files via upload
Parts:
- moved C6 48.1 mm to (157.2, 99.4), turned to 0 degrees
- moved U3 41.7 mm to (155.0, 105.0), turned to -90 degrees
- moved C5 34.6 mm to (149.4, 104.6), turned to -90 degrees
- moved F1 5.33 mm to (63.4, 99.2)
- moved J4 5.33 mm to (63.4, 110.2)
- moved H5 3.85 mm to (62.5, 64.7)
- moved PS1 3.85 mm to (74.8, 104.7)
- moved RV1 3.85 mm to (74.3, 90.2)
- moved H4 3.55 mm to (62.4, 122.4)
- moved BOOT1 1.60 mm to (179.8, 87.9)
- moved D3 1.60 mm to (168.5, 122.2)
- moved J3 1.60 mm to (149.3, 98.4)
- moved K1 1.60 mm to (138.0, 93.7)
- moved Q1 1.60 mm to (126.0, 93.4)
- moved R2 1.60 mm to (144.5, 72.4)
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- renumbered BOOT to BOOT1, EN to EN1
Connections:
- IC1 pad 10: Net-(IC1-Pad10) -> Net-(U4-Pad9)
- IC1 pad 12: Net-(IC1-Pad12) -> Net-(U4-Pad11)
- IC2 pad 10: Net-(IC2-Pad10) -> Net-(U7-Pad9)
- IC2 pad 12: Net-(IC2-Pad12) -> Net-(U7-Pad11)
- U4 pad 11: Net-(IC1-Pad10) -> Net-(U4-Pad11)
- U4 pad 9: Net-(IC1-Pad12) -> Net-(U4-Pad9)
- U5 pad 11: Net-(IC1-Pad13) -> Net-(IC1-Pad15)
- U5 pad 9: Net-(IC1-Pad15) -> Net-(IC1-Pad13)
- U7 pad 11: Net-(IC2-Pad10) -> Net-(U7-Pad11)
- U7 pad 9: Net-(IC2-Pad12) -> Net-(U7-Pad9)
- U8 pad 11: Net-(IC2-Pad13) -> Net-(IC2-Pad15)
- U8 pad 9: Net-(IC2-Pad15) -> Net-(IC2-Pad13)
Routing:
- net /SEG5_1: track 0.00 -> 101.8 mm, vias 0 -> 1
- net /SEG6_1: track 0.00 -> 97.3 mm, vias 0 -> 2
- net /SEG8_1: track 0.00 -> 97.1 mm, vias 0 -> 1
- net /SEG4_1: track 0.00 -> 95.9 mm, vias 0 -> 1
- net /SEG3_1: track 0.00 -> 85.6 mm, vias 0 -> 1
- net Net-(IC1-Pad15): track 0.00 -> 84.8 mm
- net /SEG2_1: track 0.00 -> 84.0 mm, vias 0 -> 2
- net Net-(IC1-Pad14): track 0.00 -> 83.6 mm
- net /SEG7_1: track 0.00 -> 80.4 mm, vias 0 -> 2
- net Net-(IC1-Pad13): track 0.00 -> 77.1 mm
- net /SEG1_1: track 0.12 -> 74.1 mm, vias 0 -> 2
- net /SEG2_2: track 0.00 -> 72.0 mm, vias 0 -> 1
- net /SEG8_2: track 0.00 -> 68.1 mm, vias 0 -> 1
- net /SEG7_2: track 0.00 -> 64.5 mm, vias 0 -> 1
- net /SEG1_2: track 0.00 -> 64.1 mm, vias 0 -> 1
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