File: schlum-pcb/schlum-pcb/schlum-pcb.kicad_sch (KiCad schematic)
At the start: 43 parts

Commit message: Add files via upload
Parts:
- removed D?: RED, symbol Device:LED
- removed R? (x4): 10K, symbol Device:R_US
- removed U? (x2): 2 digit 7 segments, Display_7Segment:HDSP-A151, symbol Display_Character:HDSP-7501
- removed U? (x2): 4 digit 7 segments, Display_7Segment:LTC-4627Jx, symbol Display_Character:LTC-4627JG
- added C11, C13, C14: 22u, Capacitor_SMD:C_0603_1608Metric, symbol Device:C
- added C12: 0.1u, Capacitor_SMD:C_0603_1608Metric, symbol Device:C
- added H1, H2, H3, H4, H5: MountingHole_Pad, MountingHole:MountingHole_4.3mm_M4_ISO14580_Pad, symbol Mechanical:MountingHole_Pad
- added U4, U5, U7, U8: 3_digit_7_segment, 7 segments:3 digit 7 segment, symbol 7 segments:3_digit_7_segment
- BOOT1: renamed from BOOT; footprint (none) -> Button_Switch_SMD:SW_SPST_CK_RS282G05A3
- C1, C2, C3, C5, C6: renamed from C?; footprint (none) -> Capacitor_SMD:C_0603_1608Metric
- C10, C7, C8, C9: renamed from C?; footprint (none) -> Capacitor_SMD:C_0402_1005Metric
- C4: renamed from C?; footprint (none) -> Capacitor_THT:C_Radial_D8.0mm_H11.5mm_P3.50mm
- D1: renamed from D?; footprint (none) -> Diode_SMD:D_0603_1608Metric
- D3: renamed from D?; footprint (none) -> LED_THT:LED_D5.0mm
- EN1: renamed from EN; footprint (none) -> Button_Switch_SMD:SW_SPST_CK_RS282G05A3
- F1: renamed from F?; footprint (none) -> Fuse:Fuseholder_Cylinder-5x20mm_Schurter_0031_8201_Horizontal_Open
- IC1, IC2: renamed from IC?; footprint SOIC127P1045X280-20N -> KiCad:SOIC127P1045X280-20N
- J1: renamed from J?; footprint (none) -> TerminalBlock:TerminalBlock_bornier-3_P5.08mm
- J2: renamed from J?; footprint (none) -> Connector_PinHeader_2.54mm:PinHeader_1x03_P2.54mm_Vertical
- J3: renamed from J?; footprint (none) -> Connector_PinHeader_2.54mm:PinHeader_1x04_P2.54mm_Vertical
- J4: renamed from J?; footprint (none) -> TerminalBlock:TerminalBlock_bornier-2_P5.08mm
- P1: renamed from P?; footprint (none) -> Connector_PinSocket_2.54mm:PinSocket_1x08_P2.54mm_Vertical
- R1, R2, R3: renamed from R?; footprint (none) -> Resistor_SMD:R_0402_1005Metric
- R4: renamed from R?; value 220R -> 1k; footprint (none) -> Resistor_SMD:R_0402_1005Metric
- RV1: renamed from RV?; footprint (none) -> Varistor:RV_Disc_D12mm_W5.1mm_P7.5mm
- U2: renamed from U?; footprint MODULE_ESP32-WROOM-32 -> ESP32-WROOM-32:MODULE_ESP32-WROOM-32
- gave numbers to parts that had none: 6
Connections:
- net GPIO25 is gone; now on net CLK_1: U2.10 (IO25)
- net +3.3V: now also C11.1, C12.1
- net +5V: now also C13.1, C14.1
- net CLK_1: no longer U2.12 (IO27)
- net CLK_2: now also U2.12 (IO27); no longer U2.16 (IO13)
- net GND: now also C11.2, C12.2, C13.2, C14.2, H1.1, H2.1, H3.1, H4.1, H5.1
- net MISO: now also U2.37 (IO23); no longer U2.31 (IO19)
- net MOSI: now also U2.36 (IO22); no longer U2.37 (IO23)
- net PWR_LED_C: now also D3.1 (K), R4.1
- net RA_CS: now also U2.31 (IO19); no longer U2.29 (IO5)
- net RA_RST: now also U2.33 (IO21); no longer U2.23 (IO15)
- net RFID_RST: now also U2.27 (IO16); no longer U2.14 (IO12)
- net SEG1_1: now also U4.1 (A), U5.1 (A)
- net SEG1_2: now also U7.1 (A), U8.1 (A)
- net SEG2_1: now also U4.2 (B), U5.2 (B)
- net SEG2_2: now also U7.2 (B), U8.2 (B)
- net SEG3_1: now also U4.3 (C), U5.3 (C)
- net SEG3_2: now also U7.3 (C), U8.3 (C)
- net SEG4_1: now also U4.4 (D), U5.4 (D)
- net SEG4_2: now also U7.4 (D), U8.4 (D)
- net SEG5_1: now also U4.5 (E), U5.5 (E)
- net SEG5_2: now also U7.5 (E), U8.5 (E)
- net SEG6_1: now also U4.6 (F), U5.6 (F)
- net SEG6_2: now also U7.6 (F), U8.6 (F)
- net SEG7_1: now also U4.7 (G), U5.7 (G)
- net SEG7_2: now also U7.7 (G), U8.7 (G)
- net SEG8_1: now also U4.8 (DP), U5.8 (DP)
- net SEG8_2: now also U7.8 (DP), U8.8 (DP)
- net at IC1.10 (GRID6): now also U4.11 (CA3)
- net at IC1.11 (GRID5): now also U4.10 (CA2)
- net at IC1.12 (GRID4): now also U4.9 (CA1)
- net at IC1.13 (GRID3): now also U5.11 (CA3)
- net at IC1.14 (GRID2): now also U5.10 (CA2)
- net at IC1.15 (GRID1): now also U5.9 (CA1)
- net at IC2.11 (GRID5): now also U7.10 (CA2)
- net at IC2.10 (GRID6): now also U7.11 (CA3)
- net Electrovalve_Pin: now reaches U1.2
- net Electrovalve_Pin: now also U2.14 (IO12)
- net at IC2.15 (GRID1): now also U8.9 (CA1)
- net at IC2.14 (GRID2): now also U8.10 (CA2)
- net at IC2.13 (GRID3): now also U8.11 (CA3)
- net at IC2.12 (GRID4): now also U7.9 (CA1)
- net BOOT renamed BOOT0
- net GPIO32 renamed FlowRate_PWM
Other:
- company: (none) -> Madjid
- title: (none) -> Fuel Control PCB
- moved on the sheet: C10, C7, C8, C9

Commit message: Add files via upload
Connections:
- net at U7.11 (CA3): now also IC2.12 (GRID4); no longer IC2.10 (GRID6)
- net at U7.9 (CA1): now also IC2.10 (GRID6); no longer IC2.12 (GRID4)
- net at IC1.10 (GRID6): now also U4.9 (CA1); no longer U4.11 (CA3)
- net at IC1.12 (GRID4): now also U4.11 (CA3); no longer U4.9 (CA1)
- net at IC1.13 (GRID3): now also U5.9 (CA1); no longer U5.11 (CA3)
- net at IC1.15 (GRID1): now also U5.11 (CA3); no longer U5.9 (CA1)
- net at U8.11 (CA3): now also IC2.15 (GRID1); no longer IC2.13 (GRID3)
- net at U8.9 (CA1): now also IC2.13 (GRID3); no longer IC2.15 (GRID1)
Changed lines of the file:
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@@
-    (stroke (width 0) (type default) (color 0 0 0 0))
-  )
-  (wire (pts (xy 111.76 173.99) (xy 123.19 173.99))
     (stroke (width 0) (type default) (color 0 0 0 0))
   )
@@
     (stroke (width 0) (type default) (color 0 0 0 0))
   )
+  (wire (pts (xy 118.11 119.38) (xy 118.11 123.19))
+    (stroke (width 0) (type default) (color 0 0 0 0))
+  )
   (wire (pts (xy 238.76 135.89) (xy 246.38 135.89))
     (stroke (width 0) (type default) (color 0 0 0 0))
@@
     (stroke (width 0) (type default) (color 0 0 0 0))
   )
+  (wire (pts (xy 113.665 168.91) (xy 113.665 172.72))
+    (stroke (width 0) (type default) (color 0 0 0 0))
+  )
   (polyline (pts (xy 170.18 146.05) (xy 19.05 146.05))
     (stroke (width 0) (type default) (color 0 0 0 0))
   )
-  (wire (pts (xy 85.725 185.42) (xy 85.725 173.99))
-    (stroke (width 0) (type default) (color 0 0 0 0))
-  )
   (wire (pts (xy 86.36 85.09) (xy 89.535 85.09))
     (stroke (width 0) (type default) (color 0 0 0 0))
@@
     (stroke (width 0) (type default) (color 0 0 0 0))
   )
+  (wire (pts (xy 116.205 173.99) (xy 111.76 173.99))
+    (stroke (width 0) (type default) (color 0 0 0 0))
+  )
   (wire (pts (xy 123.19 179.07) (xy 88.265 179.07))
     (stroke (width 0) (type default) (color 0 0 0 0))
@@
     (stroke (width 0) (type default) (color 0 0 0 0))
   )
-  (wire (pts (xy 111.76 119.38) (xy 123.19 119.38))
-    (stroke (width 0) (type default) (color 0 0 0 0))
-  )
   (wire (pts (xy 118.11 161.29) (xy 123.19 161.29))
     (stroke (width 0) (type default) (color 0 0 0 0))
@@
     (stroke (width 0) (type default) (color 0 0 0 0))
   )
-  (wire (pts (xy 123.19 127) (xy 89.535 127))
-    (stroke (width 0) (type default) (color 0 0 0 0))
-  )
   (wire (pts (xy 138.43 85.09) (xy 138.43 87.63))
     (stroke (width 0) (type default) (color 0 0 0 0))
@@
     (stroke (width 0) (type default) (color 0 0 0 0))
   )
-  (wire (pts (xy 89.535 127) (xy 89.535 119.38))
-    (stroke (width 0) (type default) (color 0 0 0 0))
-  )
   (wire (pts (xy 123.19 74.93) (xy 125.73 74.93))
     (stroke (width 0) (type default) (color 0 0 0 0))
@@
     (stroke (width 0) (type default) (color 0 0 0 0))
   )
+  (wire (pts (xy 90.17 176.53) (xy 90.17 173.99))
+    (stroke (width 0) (type default) (color 0 0 0 0))
+  )
   (wire (pts (xy 238.76 148.59) (xy 246.38 148.59))
     (stroke (width 0) (type default) (color 0 0 0 0))
@@
     (stroke (width 0) (type default) (color 0 0 0 0))
   )
+  (wire (pts (xy 116.205 168.91) (xy 116.205 173.99))
+    (stroke (width 0) (type default) (color 0 0 0 0))
+  )
   (wire (pts (xy 97.79 87.63) (xy 110.49 87.63))
     (stroke (width 0) (type default) (color 0 0 0 0))
@@
     (stroke (width 0) (type default) (color 0 0 0 0))
   )
+  (wire (pts (xy 123.19 168.91) (xy 116.205 168.91))
+    (stroke (width 0) (type default) (color 0 0 0 0))
+  )
+  (wire (pts (xy 113.03 123.19) (xy 113.03 124.46))
+    (stroke (width 0) (type default) (color 0 0 0 0))
+  )
   (wire (pts (xy 110.49 87.63) (xy 123.19 87.63))
     (stroke (width 0) (type default) (color 0 0 0 0))
@@
     (stroke (width 0) (type default) (color 0 0 0 0))
   )
-  (wire (pts (xy 158.75 135.89) (xy 85.725 135.89))
-    (stroke (width 0) (type default) (color 0 0 0 0))
-  )
   (wire (pts (xy 123.19 72.39) (xy 123.19 74.93))
     (stroke (width 0) (type default) (color 0 0 0 0))
@@
     (stroke (width 0) (type default) (color 0 0 0 0))
   )
-  (wire (pts (xy 90.17 168.91) (xy 85.725 168.91))
-    (stroke (width 0) (type default) (color 0 0 0 0))
-  )
   (polyline (pts (xy 170.18 99.06) (xy 170.18 110.49))
     (stroke (width 0) (type default) (color 0 0 0 0))
@@
     (stroke (width 0) (type default) (color 0 0 0 0))
   )
+  (wire (pts (xy 123.19 172.72) (xy 123.19 173.99))
+    (stroke (width 0) (type default) (color 0 0 0 0))
+  )
   (polyline (pts (xy 140.97 66.04) (xy 140.97 95.25))
     (stroke (width 0) (type default) (color 0 0 0 0))
@@
     (stroke (width 0) (type default) (color 0 0 0 0))
   )
+  (wire (pts (xy 123.19 119.38) (xy 118.11 119.38))
+    (stroke (width 0) (type default) (color 0 0 0 0))
+  )
   (wire (pts (xy 162.56 114.3) (xy 158.75 114.3))
     (stroke (width 0) (type default) (color 0 0 0 0))
@@
     (stroke (width 0) (type default) (color 0 0 0 0))
   )
+  (wire (pts (xy 87.63 185.42) (xy 87.63 168.91))
+    (stroke (width 0) (type default) (color 0 0 0 0))
+  )
   (wire (pts (xy 118.11 163.83) (xy 123.19 163.83))
     (stroke (width 0) (type default) (color 0 0 0 0))
@@
     (stroke (width 0) (type default) (color 0 0 0 0))
   )
+  (wire (pts (xy 113.665 172.72) (xy 123.19 172.72))
+    (stroke (width 0) (type default) (color 0 0 0 0))
+  )
   (wire (pts (xy 91.44 119.38) (xy 96.52 119.38))
     (stroke (width 0) (type default) (color 0 0 0 0))
@@
     (stroke (width 0) (type default) (color 0 0 0 0))
   )
+  (wire (pts (xy 111.76 168.91) (xy 113.665 168.91))
+    (stroke (width 0) (type default) (color 0 0 0 0))
+  )
   (wire (pts (xy 47.625 186.69) (xy 47.625 185.42))
     (stroke (width 0) (type default) (color 0 0 0 0))
@@
     (stroke (width 0) (type default) (color 0 0 0 0))
   )
-  (wire (pts (xy 158.75 185.42) (xy 85.725 185.42))
-    (stroke (width 0) (type default) (color 0 0 0 0))
-  )
   (wire (pts (xy 135.255 36.195) (xy 135.255 40.64))
     (stroke (width 0) (type default) (color 0 0 0 0))
@@
     (stroke (width 0) (type default) (color 0 0 0 0))
   )
+  (wire (pts (xy 87.63 168.91) (xy 85.725 168.91))
+    (stroke (width 0) (type default) (color 0 0 0 0))
+  )
   (wire (pts (xy 211.455 68.58) (xy 215.9 68.58))
     (stroke (width 0) (type default) (color 0 0 0 0))
@@
     (stroke (width 0) (type default) (color 0 0 0 0))
   )
+  (wire (pts (xy 114.935 119.38) (xy 111.76 119.38))
+    (stroke (width 0) (type default) (color 0 0 0 0))
+  )
   (wire (pts (xy 264.16 71.12) (xy 256.54 71.12))
     (stroke (width 0) (type default) (color 0 0 0 0))
@@
     (stroke (width 0) (type default) (color 0 0 0 0))
   )
-  (wire (pts (xy 111.76 168.91) (xy 123.19 168.91))
-    (stroke (width 0) (type default) (color 0 0 0 0))
-  )
   (wire (pts (xy 162.56 119.38) (xy 158.75 119.38))
     (stroke (width 0) (type default) (color 0 0 0 0))
   )
+  (wire (pts (xy 85.725 127) (xy 123.19 127))
+    (stroke (width 0) (type default) (color 0 0 0 0))
+  )
   (wire (pts (xy 65.405 114.3) (xy 70.485 114.3))
     (stroke (width 0) (type default) (color 0 0 0 0))
@@
     (stroke (width 0) (type default) (color 0 0 0 0))
   )
+  (wire (pts (xy 123.19 124.46) (xy 114.935 124.46))
+    (stroke (width 0) (type default) (color 0 0 0 0))
+  )
   (wire (pts (xy 118.11 114.3) (xy 123.19 114.3))
     (stroke (width 0) (type default) (color 0 0 0 0))
@@
     (stroke (width 0) (type default) (color 0 0 0 0))
   )
+  (wire (pts (xy 85.725 124.46) (xy 85.725 127))
+    (stroke (width 0) (type default) (color 0 0 0 0))
+  )
   (wire (pts (xy 162.56 168.91) (xy 158.75 168.91))
     (stroke (width 0) (type default) (color 0 0 0 0))
@@
     (stroke (width 0) (type default) (color 0 0 0 0))
   )
+  (wire (pts (xy 90.17 173.99) (xy 85.725 173.99))
+    (stroke (width 0) (type default) (color 0 0 0 0))
+  )
   (polyline (pts (xy 28.575 95.25) (xy 76.835 95.25))
     (stroke (width 0) (type default) (color 0 0 0 0))
@@
     (stroke (width 0) (type default) (color 0 0 0 0))
   )
+  (wire (pts (xy 158.75 135.89) (xy 89.535 135.89))
+    (stroke (width 0) (type default) (color 0 0 0 0))
+  )
   (wire (pts (xy 111.76 171.45) (xy 123.19 171.45))
     (stroke (width 0) (type default) (color 0 0 0 0))
@@
     (stroke (width 0) (type default) (color 0 0 0 0))
   )
-  (wire (pts (xy 85.725 135.89) (xy 85.725 124.46))
-    (stroke (width 0) (type default) (color 0 0 0 0))
-  )
   (wire (pts (xy 123.19 74.93) (xy 118.11 74.93))
     (stroke (width 0) (type default) (color 0 0 0 0))
@@
     (stroke (width 0) (type default) (color 0 0 0 0))
   )
+  (wire (pts (xy 118.11 123.19) (xy 113.03 123.19))
+    (stroke (width 0) (type default) (color 0 0 0 0))
+  )
   (wire (pts (xy 59.69 82.55) (xy 66.04 82.55))
     (stroke (width 0) (type default) (color 0 0 0 0))
@@
     (stroke (width 0) (type default) (color 0 0 0 0))
   )
+  (wire (pts (xy 89.535 119.38) (xy 89.535 135.89))
+    (stroke (width 0) (type default) (color 0 0 0 0))
+  )
   (wire (pts (xy 65.405 173.99) (xy 70.485 173.99))
     (stroke (width 0) (type default) (color 0 0 0 0))
@@
     (stroke (width 0) (type default) (color 0 0 0 0))
   )
-  (wire (pts (xy 111.76 124.46) (xy 123.19 124.46))
+  (wire (pts (xy 114.935 124.46) (xy 114.935 119.38))
     (stroke (width 0) (type default) (color 0 0 0 0))
   )
@@
     (stroke (width 0) (type default) (color 0 0 0 0))
   )
+  (wire (pts (xy 158.75 185.42) (xy 87.63 185.42))
+    (stroke (width 0) (type default) (color 0 0 0 0))
+  )
+  (wire (pts (xy 113.03 124.46) (xy 111.76 124.46))
+    (stroke (width 0) (type default) (color 0 0 0 0))
+  )
   (wire (pts (xy 93.98 24.13) (xy 115.57 24.13))
     (stroke (width 0) (type default) (color 0 0 0 0))
@@
     (stroke (width 0) (type default) (color 0 0 0 0))
   )
-  (wire (pts (xy 90.17 176.53) (xy 90.17 168.91))
-    (stroke (width 0) (type default) (color 0 0 0 0))
-  )
